File: Advanced-PCB-Workshop.kicad_pcb (KiCad board)
At the start: 4 copper layers, 39.9 x 39.5 mm, 36 parts, among them J1 USB_C_Receptacle_USB2.0_14P, J2 Conn_01x03_Pin, J3 Conn_01x14_Socket, J4 Conn_01x14_Socket, SW1 SW_Nidec_CAS-120A1, SW2 SW_Push, U1 RP2040, U2 W25Q128JVS, U3 AMS1117-3.3, Y1 ABM8-272-T3

Commit message: Finish Template Board
Routing:
- net QSPI_SD3: track 1.41 -> 0.67 mm
Other:
- copper layers 4 -> 2
Changed lines of the file:
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@@
 	(layers
 		(0 "F.Cu" signal)
-		(4 "In1.Cu" signal)
-		(6 "In2.Cu" signal)
 		(2 "B.Cu" signal)
 		(9 "F.Adhes" user "F.Adhesive")
@@
 			)
 			(layer "dielectric 1"
-				(type "prepreg")
-				(thickness 0.1)
-				(material "FR4")
-				(epsilon_r 4.5)
-				(loss_tangent 0.02)
-			)
-			(layer "In1.Cu"
-				(type "copper")
-				(thickness 0.035)
-			)
-			(layer "dielectric 2"
 				(type "core")
-				(thickness 1.24)
-				(material "FR4")
-				(epsilon_r 4.5)
-				(loss_tangent 0.02)
-			)
-			(layer "In2.Cu"
-				(type "copper")
-				(thickness 0.035)
-			)
-			(layer "dielectric 3"
-				(type "prepreg")
-				(thickness 0.1)
+				(thickness 1.51)
 				(material "FR4")
 				(epsilon_r 4.5)
@@
 		(tags "capacitor")
 		(property "Reference" "C3"
-			(at -0.98 -1.37 0)
+			(at -1.25 0 0)
 			(layer "F.SilkS")
 			(effects
 				(font
-					(size 1 1)
-					(thickness 0.15)
+					(size 0.5 0.5)
+					(thickness 0.125)
 				)
 			)
@@
 		(tags "capacitor")
 		(property "Reference" "C6"
-			(at -1.3 1.1 180)
+			(at -1.28 0.09 180)
 			(layer "F.SilkS")
 			(effects
 				(font
-					(size 1 1)
-					(thickness 0.15)
+					(size 0.5 0.5)
+					(thickness 0.125)
 				)
 			)
@@
 			(effects
 				(font
-					(size 1 1)
-					(thickness 0.15)
+					(size 0.5 0.5)
+					(thickness 0.125)
 				)
 			)
@@
 		(tags "capacitor")
 		(property "Reference" "C2"
-			(at 0.02 1.13 90)
+			(at 0.19 1.11 90)
 			(layer "F.SilkS")
 			(effects
@@
 	)
 	(gr_text "D18"
-		(at 150.62 118.14 0)
+		(at 150.61 117.89 0)
 		(layer "F.SilkS")
 		(effects
@@
 		(width 0.1)
 		(layer "F.Cu")
-		(net 48)
-	)
-	(segment
-		(start 131.3725 107.8525)
-		(end 131.3725 107.1125)
-		(width 0.1)
-		(layer "F.Cu")

Commit message: Completed Board
Parts:
- moved SW1 10.3 mm to (123.4, 85.3), turned to -90 degrees
- moved R3 3.37 mm to (124.9, 96.7), turned to -90 degrees
- moved C15 1.65 mm to (127.6, 107.3), turned to -90 degrees
- moved C3 1.56 mm to (135.7, 104.9)
- moved C4 1.50 mm to (137.2, 105.9)
- moved C1 1.44 mm to (133.8, 117.9)
- moved C16 1.29 mm to (132.7, 117.9)
- moved C13 0.91 mm to (130.5, 117.8)
- moved C14 0.90 mm to (131.7, 117.9)
- moved C10 0.84 mm to (137.2, 107.0)
- moved R6 0.74 mm to (131.3, 95.5)
- moved R7 0.73 mm to (134.7, 95.5)
- moved C9 0.52 mm to (126.3, 112.1)
- moved C7 0.46 mm to (137.2, 108.2)
- moved C8 0.38 mm to (137.6, 112.3)
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Connections:
- net /USBDM renamed /USBDN
Routing:
- net +5V: track 0.00 -> 32.6 mm, vias 0 -> 2
- net D0: track 0.00 -> 32.5 mm
- net D1: track 0.00 -> 30.4 mm
- net D2: track 0.00 -> 28.3 mm
- net A3: track 0.00 -> 26.2 mm, vias 0 -> 1
- net D3: track 0.00 -> 26.1 mm
- net A2: track 0.00 -> 24.3 mm, vias 0 -> 1
- net D4: track 0.00 -> 24.0 mm
- net A1: track 0.00 -> 22.4 mm, vias 0 -> 1
- net D5: track 0.00 -> 21.9 mm
- net D25: track 0.00 -> 21.7 mm
- net A0: track 0.00 -> 21.7 mm, vias 0 -> 1
- net IOVDD: track 1.54 -> 22.8 mm, vias 0 -> 21
- net D24: track 0.00 -> 20.2 mm
- net D6: track 0.00 -> 19.8 mm
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- added copper zone on B.Cu, net GND
- added copper zone on F.Cu, net GND
- added copper zone on In1.Cu, net GND
- added copper zone on In2.Cu, net IOVDD
Other:
- copper layers 2 -> 4
