File: Advanced-PCB-Workshop.kicad_pcb (KiCad board)
At the start: 2 copper layers, 39.9 x 39.5 mm, 36 parts, among them J1 USB_C_Receptacle_USB2.0_14P, J2 Conn_01x03_Pin, J3 Conn_01x14_Socket, J4 Conn_01x14_Socket, SW1 SW_Nidec_CAS-120A1, SW2 SW_Push, U1 RP2040, U2 W25Q128JVS, U3 AMS1117-3.3, Y1 ABM8-272-T3

Commit message: Final Template
Parts:
- moved SW1 10.9 mm to (123.0, 84.7), turned to -90 degrees
- moved R4 3.33 mm to (123.2, 97.1), turned to 0 degrees
- moved C4 1.93 mm to (137.6, 106.0)
- moved C9 1.33 mm to (125.4, 112.3)
- moved C3 1.16 mm to (135.3, 105.2)
- moved C15 1.13 mm to (125.5, 108.7)
- moved C10 1.03 mm to (137.6, 107.3)
- moved R3 0.79 mm to (123.2, 98.7)
- moved C7 0.49 mm to (137.6, 108.4)
- moved C8 0.46 mm to (137.6, 112.3)
- moved C2 0.16 mm to (131.0, 105.2)
- moved C6 0.16 mm to (132.1, 105.2)
- moved C5 0.16 mm to (133.1, 105.2)
- moved R2 0.11 mm to (125.8, 90.3)
Routing:
- net IOVDD: track 1.54 -> 0.23 mm

Commit message: Final Template v1.1.1
Connections:
- net /USBDM renamed /USBDN
Changed lines of the file:
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@@
 	(net 51 "Net-(J1-CC1)")
 	(net 52 "/USBDP")
-	(net 53 "/USBDM")
+	(net 53 "/USBDN")
 	(footprint "Capacitor_SMD:C_0402_1005Metric"
 		(layer "F.Cu")
@@
 			(layers "F.Cu" "F.Mask" "F.Paste")
 			(roundrect_rratio 0.25)
-			(net 53 "/USBDM")
+			(net 53 "/USBDN")
 			(pinfunction "USB_DM")
 			(pintype "bidirectional")
@@
 			(layers "F.Cu" "F.Mask" "F.Paste")
 			(roundrect_rratio 0.25)
-			(net 53 "/USBDM")
+			(net 53 "/USBDN")
 			(pintype "passive")
 		)

Commit message: Final Template v1.2.0
Parts:
- moved R6 0.81 mm to (130.7, 95.7)
- moved R7 0.81 mm to (134.1, 95.7)
Changed lines of the file:
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@@
 	(footprint "Resistor_SMD:R_0603_1608Metric_Pad0.98x0.95mm_HandSolder"
 		(layer "F.Cu")
-		(at 134.2675 94.93 180)
+		(at 134.1275 95.73 180)
 		(descr "Resistor SMD 0603 (1608 Metric), square (rectangular) end terminal, IPC-7351 nominal with elongated pad for handsoldering. (Body size source: IPC-SM-782 page 72, https://www.pcb-3d.com/wordpress/wp-content/uploads/ipc-sm-782a_amendment_1_and_2.pdf), generated with kicad-footprint-generator")
 		(tags "resistor handsolder")
 		(property "Reference" "R7"
-			(at 0 -1.43 0)
+			(at -2.6025 -0.06 0)
 			(layer "F.SilkS")
 			(effects
@@
 	(footprint "Resistor_SMD:R_0603_1608Metric_Pad0.98x0.95mm_HandSolder"
 		(layer "F.Cu")
-		(at 130.83 94.94)
+		(at 130.69 95.74)
 		(descr "Resistor SMD 0603 (1608 Metric), square (rectangular) end terminal, IPC-7351 nominal with elongated pad for handsoldering. (Body size source: IPC-SM-782 page 72, https://www.pcb-3d.com/wordpress/wp-content/uploads/ipc-sm-782a_amendment_1_and_2.pdf), generated with kicad-footprint-generator")
 		(tags "resistor handsolder")
