File: Advanced-PCB-Workshop.kicad_sch (KiCad schematic)
At the start: 33 parts, among them J1 USB_C_Receptacle_USB2.0_14P, J2 Conn_01x03_Pin, J3 Conn_01x14_Socket, J4 Conn_01x14_Socket, SW1 SW_Nidec_CAS-120A1, SW2 SW_Push, U1 RP2040, U2 W25Q128JVS, U3 AMS1117-3.3, Y1 ABM8-272-T3

Commit message: Final Template v1.1
Connections:
- net USBDM renamed USBDN
Changed lines of the file:
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@@
 		)
 	)
-	(label "USBDM"
+	(label "USBDN"
 		(at 88.9 91.44 0)
 		(effects
